File: Keyboard.kicad_pcb (KiCad board)
At the start: 2 copper layers, 138.9 x 76.2 mm, 56 parts, among them SW1 SW_Push, U1 ATmega32U4-AU, Y1 16MHz

Commit message: really bad traces but atleast i hope it works
doesn't connect key matrix to the mcu
Parts:
- moved SW1 24.8 mm to (73.1, 98.4)
- moved C7 5.65 mm to (77.8, 108.9), turned to 90 degrees
- moved R1 5.56 mm to (81.0, 93.8)
- moved F1 2.51 mm to (64.3, 104.6)
- moved R2 2.51 mm to (69.8, 104.1)
- moved R3 2.51 mm to (67.5, 104.1)
- moved C3 1.23 mm to (75.4, 103.3)
- turned D11 to 90 degrees
Routing:
- net GND: track 0.00 -> 138.9 mm
- net +5V: track 0.00 -> 95.0 mm, vias 0 -> 8
- net row3: track 0.00 -> 78.5 mm
- net row0: track 0.00 -> 78.5 mm
- net row1: track 0.00 -> 78.5 mm
- net row2: track 0.00 -> 78.4 mm
- net col0: track 0.00 -> 54.4 mm
- net col4: track 0.00 -> 54.4 mm
- net col3: track 0.00 -> 54.4 mm
- net col2: track 0.00 -> 54.4 mm
- net col1: track 0.00 -> 54.4 mm
- net Net-(R1-Pad2): track 0.00 -> 22.2 mm
- net Net-(R3-Pad1): track 0.00 -> 14.3 mm
- net Net-(C2-Pad2): track 0.00 -> 12.3 mm
- net Net-(R2-Pad1): track 0.00 -> 11.9 mm
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Other:
- net class Default: trace_width 0.25 -> 0.254
- net class Power added: clearance 0.2, trace_width 0.381, via_dia 0.8, via_drill 0.4

Commit message: terribly connected key matrix
Connections:
- U1 pad 25: Net-(U1-Pad25) -> col0
- U1 pad 26: Net-(U1-Pad26) -> col1
- U1 pad 27: Net-(U1-Pad27) -> col2
- U1 pad 28: Net-(U1-Pad28) -> col3
- U1 pad 29: Net-(U1-Pad29) -> col4
- U1 pad 30: Net-(U1-Pad30) -> row0
- U1 pad 31: Net-(U1-Pad31) -> row1
- U1 pad 32: Net-(U1-Pad32) -> row2
- U1 pad 39: Net-(U1-Pad39) -> row3
Routing:
- net col2: track 54.4 -> 231.1 mm
- net col4: track 54.4 -> 153.8 mm
- net row3: track 78.5 -> 161.5 mm
- net col3: track 54.4 -> 135.6 mm, vias 0 -> 1
- net row2: track 78.4 -> 122.5 mm
- net row1: track 78.5 -> 122.4 mm, vias 0 -> 4
- net col1: track 54.4 -> 92.4 mm
- net row0: track 78.5 -> 109.3 mm, vias 0 -> 4
- net col0: track 54.4 -> 73.3 mm
- net Net-(USB1-Pad6): track 0.00 -> 16.3 mm

Commit message: add watermark if you just wanna copy me without knowing anything
Routing:
- net +5V: track 95.0 -> 99.8 mm
- added copper zone on B.Cu, net GND
Changed lines of the file:
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@@
     (thickness 1.6)
     (drawings 8)
-    (tracks 406)
+    (tracks 412)
     (zones 0)
     (modules 56)
@@
   (segment (start 81.86275 108.09375) (end 82.51875 108.09375) (width 0.381) (layer B.Cu) (net 5))
   (segment (start 80.84099 107.07199) (end 81.86275 108.09375) (width 0.381) (layer B.Cu) (net 5))
-  (segment (start 77.06853 107.07199) (end 80.84099 107.07199) (width 0.381) (layer B.Cu) (net 5))
   (segment (start 75.69375 108.44677) (end 77.06853 107.07199) (width 0.381) (layer B.Cu) (net 5))
   (segment (start 75.69375 109.825) (end 75.69375 108.44677) (width 0.381) (layer B.Cu) (net 5))
@@
   (segment (start 84.11875 94.4375) (end 84.11875 95.23125) (width 0.381) (layer B.Cu) (net 5))
   (segment (start 84.11875 95.23125) (end 84.11875 96.69375) (width 0.381) (layer B.Cu) (net 5))
+  (segment (start 80.9625 94.74375) (end 80.9625 96.8375) (width 0.381) (layer B.Cu) (net 5))
+  (segment (start 80.9625 96.8375) (end 78.58125 96.8375) (width 0.381) (layer B.Cu) (net 5))
+  (segment (start 78.648524 107.055004) (end 78.66551 107.07199) (width 0.381) (layer B.Cu) (net 5))
+  (segment (start 78.648524 106.790948) (end 78.648524 107.055004) (width 0.381) (layer B.Cu) (net 5))
+  (segment (start 77.06853 107.07199) (end 78.66551 107.07199) (width 0.381) (layer B.Cu) (net 5))
+  (segment (start 78.66551 107.07199) (end 80.84099 107.07199) (width 0.381) (layer B.Cu) (net 5))
   (segment (start 117.26875 95.1875) (end 119.85625 95.1875) (width 0.254) (layer B.Cu) (net 6))
   (segment (start 114.41875 92.3375) (end 117.26875 95.1875) (width 0.254) (layer B.Cu) (net 6))
@@
   (segment (start 119.00225 118.2415) (end 119.70625 117.5375) (width 0.254) (layer B.Cu) (net 13))
   (segment (start 110.951624 118.2415) (end 119.00225 118.2415) (width 0.254) (layer B.Cu) (net 13))
-  (segment (start 92.21875 104.79375) (end 97.503874 104.79375) (width 0.254) (layer B.Cu) (net 13))
   (via (at 110.933013 118.286801) (size 0.8) (drill 0.4) (layers F.Cu B.Cu) (net 13))
   (segment (start 110.951624 118.2415) (end 110.951624 118.26819) (width 0.254) (layer B.Cu) (net 13))
@@
   (segment (start 101.6 115.09375) (end 99.21875 112.7125) (width 0.254) (layer F.Cu) (net 13))
   (segment (start 99.21875 112.7125) (end 99.21875 104.775) (width 0.254) (layer F.Cu) (net 13))
-  (segment (start 99.21875 104.775) (end 97.63125 104.775) (width 0.254) (layer B.Cu) (net 13))
+  (segment (start 97.503874 104.79375) (end 92.21875 104.79375) (width 0.254) (layer B.Cu) (net 13))
+  (segment (start 99.21875 104.775) (end 97.522624 104.775) (width 0.254) (layer B.Cu) (net 13))
+  (segment (start 97.522624 104.775) (end 97.503874 104.79375) (width 0.254) (layer B.Cu) (net 13))
   (segment (start 136.31875 114.2375) (end 138.90625 114.2375) (width 0.254) (layer B.Cu) (net 14))
   (segment (start 133.46875 111.3875) (end 136.31875 114.2375) (width 0.254) (layer B.Cu) (net 14))
@@
   (segment (start 71.11875 88.9) (end 71.11875 93.4) (width 0.254) (layer B.Cu) (net 59))
   (segment (start 63.81875 93.4) (end 63.81875 88.9) (width 0.254) (layer B.Cu) (net 59))
+  (zone (net 2) (net_name GND) (layer B.Cu) (hatch edge 0.508)
+    (connect_pads (clearance 0.508))
+    (min_thickness 0.254)
+    (fill yes (arc_segments 32) (thermal_gap 0.508) (thermal_bridge_width 0.508))
+    (polygon
+      (pts
+        (xy 81.75625 97.63125) (xy 81.75625 107.15625) (xy 91.28125 107.15625) (xy 91.28125 97.63125)
+      )
+    )
+  )
+  (zone (net 2) (net_name GND) (layer B.Cu) (hatch edge 0.508)
+    (connect_pads (clearance 0.508))
+    (min_thickness 0.254)
+    (fill yes (arc_segments 32) (thermal_gap 0.508) (thermal_bridge_width 0.508))
+    (polygon
+      (pts
+        (xy 76.99375 87.3125) (xy 76.99375 93.6625) (xy 76.99375 95.25) (xy 92.86875 95.25) (xy 92.86875 87.3125)
+      )
+    )
+  )
+  (zone (net 2) (net_name GND) (layer B.Cu) (hatch edge 0.508)
+    (connect_pads (clearance 0.508))
+    (min_thickness 0.254)
+    (fill yes (arc_segments 32) (thermal_gap 0.508) (thermal_bridge_width 0.508))
+    (polygon
+      (pts
+        (xy 72.23125 87.3125) (xy 72.23125 96.04375) (xy 62.70625 96.04375) (xy 62.70625 87.3125)
+      )
+    )
+  )
 )

Commit message: Add Gerbers & Drill files
Other:
- board text added: "github.com/alexfeed1990/Macro-Pad"
Changed lines of the file:
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@@
   (general
     (thickness 1.6)
-    (drawings 8)
+    (drawings 9)
     (tracks 412)
     (zones 0)
@@
     (visible_elements FFFFFF7F)
     (pcbplotparams
-      (layerselection 0x010fc_ffffffff)
-      (usegerberextensions false)
+      (layerselection 0x010f0_ffffffff)
+      (usegerberextensions true)
       (usegerberattributes false)
       (usegerberadvancedattributes false)
@@
       (plotinvisibletext false)
       (padsonsilk false)
-      (subtractmaskfromsilk false)
+      (subtractmaskfromsilk true)
       (outputformat 1)
       (mirror false)
-      (drillshape 1)
+      (drillshape 0)
       (scaleselection 1)
-      (outputdirectory ""))
+      (outputdirectory "Gerbers/"))
   )
   (net 0 "")
@@
     )
   )
+  (gr_text github.com/alexfeed1990/Macro-Pad (at 76.99375 160.3375) (layer F.SilkS)
+    (effects (font (size 1 1) (thickness 0.15) italic))
+  )
   (gr_line (start 61.9125 163.5125) (end 194.46875 163.5125) (layer Edge.Cuts) (width 0.05))
